File: ProtosuitDevBoard/ProtosuitDevBoard.kicad_pcb (KiCad board)
At the start: 2 copper layers, 31 parts, among them J1 XT60 IN, J10 Left Ear, J11 Right Ear, J12 Microphone input, J13 Display I2C, J14 Extra I2C, J15 Boop Sensor I2C, J16 Gyroscope I2C, J2 RPi Out, J3 Front Left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

Commit message: Final dev board
Parts:
- added J17: DHT22 sensor, Connector_JST:JST_XH_B3B-XH-A_1x03_P2.50mm_Vertical, F.Cu at (154.0, 65.0)
- added Q1: 2N3904, Package_TO_SOT_THT:TO-92_Inline, F.Cu at (158.5, 100.0)
- added R1: 4k7, Resistor_THT:R_Axial_DIN0207_L6.3mm_D2.5mm_P2.54mm_Vertical, F.Cu at (150.0, 90.5)
- added R2: 2k2, Resistor_THT:R_Axial_DIN0207_L6.3mm_D2.5mm_P2.54mm_Vertical, F.Cu at (166.0, 93.5)
- added R3: 100k, Resistor_THT:R_Axial_DIN0207_L6.3mm_D2.5mm_P2.54mm_Vertical, F.Cu at (164.0, 98.5)
- added R4: 10k, Resistor_THT:R_Axial_DIN0207_L6.3mm_D2.5mm_P2.54mm_Vertical, F.Cu at (150.0, 96.5)
- added U7: MPU6050 Gyroscope, Aliexpress:GYRO_MPU6050, F.Cu at (136.7, 68.5)
- J1: value XT60 IN -> PWR IN
- J16: value Gyroscope I2C -> FAN; footprint Connector_JST:JST_XH_B4B-XH-A_1x04_P2.50mm_Vertical -> Connector:FanPinHeader_1x04_P2.54mm_Vertical_No_Via
- U3: value Teensy4.0 -> Teensy 4.0; footprint teensy:Teensy40 -> teensy:Teensy40_minimal_pins
- U4: value ESP32 Mini -> Wemos D1 Mini ESP32
- U5: value Level Shifter TXS0108E -> Level Shifter LED matrix
- U6: value Level Shifter TXS0108E -> Level Shifter LED strips
- moved J7 154.6 mm to (213.0, 92.0), turned to 50 degrees
- moved RV5 139.3 mm to (211.3, 82.1), turned to 50 degrees
- moved J6 110.9 mm to (164.2, 141.0)
- moved J4 101.2 mm to (180.0, 131.3), turned to 50 degrees
- moved J10 96.6 mm to (96.0, 141.0), turned to 0 degrees
- moved J3 96.5 mm to (147.0, 141.0), turned to 0 degrees
- moved RV1 95.7 mm to (171.1, 133.0)
- moved J9 87.3 mm to (191.0, 118.3), turned to 50 degrees
- moved RV4 86.8 mm to (154.1, 133.0), turned to 0 degrees
- moved J8 86.8 mm to (113.0, 141.0), turned to 0 degrees
- moved U4 82.4 mm to (180.0, 63.3)
- moved RV8 82.2 mm to (106.0, 133.0), turned to 0 degrees
- moved U6 82.0 mm to (182.5, 94.2), turned to -90 degrees
- moved RV3 80.0 mm to (180.6, 118.1), turned to 50 degrees
- moved RV6 74.0 mm to (121.1, 133.0), turned to 0 degrees
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Connections:
- J1 pad 1: Net-(J1-Pin_1) -> GND
- J10 pad 1: Net-(J10-Pin_1) -> GND
- J10 pad 2: Net-(J10-Pin_2) -> +5V
- J11 pad 1: Net-(J10-Pin_1) -> GND
- J11 pad 2: Net-(J10-Pin_2) -> +5V
- J12 pad 1: Net-(J12-Pin_1) -> GND
- J13 pad 1: Net-(J10-Pin_1) -> GND
- J14 pad 1: Net-(J10-Pin_1) -> GND
- J15 pad 1: Net-(J15-Pin_1) -> GND
- J15 pad 2: Net-(J15-Pin_2) -> Net-(J12-Pin_2)
- J16 pad 1: Net-(J15-Pin_1) -> GND
- J16 pad 2: Net-(J15-Pin_2) -> +5V
- J16 pad 3: Net-(J15-Pin_3) -> Net-(J16-Pin_3)
- J16 pad 4: Net-(J15-Pin_4) -> Net-(J16-Pin_4)
- J2 pad 1: Net-(J2-Pin_1) -> GND
- J3 pad 1: Net-(J10-Pin_1) -> GND
- J3 pad 2: Net-(J10-Pin_2) -> +5V
- J4 pad 1: Net-(J10-Pin_1) -> GND
- J4 pad 2: Net-(J10-Pin_2) -> +5V
- J5 pad 1: Net-(J10-Pin_1) -> GND
- J5 pad 2: Net-(J10-Pin_2) -> +5V
- J6 pad 1: Net-(J10-Pin_1) -> GND
- J6 pad 2: Net-(J10-Pin_2) -> +5V
- J7 pad 1: Net-(J10-Pin_1) -> GND
- J7 pad 2: Net-(J10-Pin_2) -> +5V
- J8 pad 1: Net-(J10-Pin_1) -> GND
- J8 pad 2: Net-(J10-Pin_2) -> +5V
- J9 pad 1: Net-(J10-Pin_1) -> GND
- J9 pad 2: Net-(J10-Pin_2) -> +5V
- U1 pad 2: Net-(J1-Pin_1) -> GND
- U1 pad 4: Net-(J2-Pin_1) -> GND
- U2 pad 2: Net-(J1-Pin_1) -> GND
- U2 pad 3: Net-(J10-Pin_2) -> +5V
- U2 pad 4: Net-(J10-Pin_1) -> GND
- U3 pad 1: Net-(J15-Pin_1) -> GND
- U3 pad 31: unconnected-(U3-3V3-Pad31) -> Net-(J12-Pin_2)
- U3 pad 32: Net-(J10-Pin_1) -> GND
- U3 pad 33: Net-(J10-Pin_2) -> +5V
- U4 pad 1: Net-(U6-GND) -> GND
- U4 pad 27: Net-(J10-Pin_1) -> GND
- U4 pad 28: Net-(J10-Pin_2) -> +5V
- U4 pad 31: unconnected-(U4-GND-Pad31) -> GND
- U4 pad 32: unconnected-(U4-IO27-Pad32) -> Net-(J17-Pin_3)
- U4 pad 4: unconnected-(U4-IO35-Pad4) -> Net-(J16-Pin_3)
- U4 pad 5: unconnected-(U4-IO33-Pad5) -> Net-(U4-IO33)
- U5 pad 1: Net-(J15-Pin_2) -> Net-(J12-Pin_2)
- U5 pad 11: Net-(J10-Pin_2) -> +5V
- U5 pad 20: Net-(J15-Pin_1) -> GND
- U6 pad 11: Net-(J10-Pin_2) -> +5V
- U6 pad 20: Net-(U6-GND) -> GND
Routing:
- net Net-(J12-Pin_2): track 0.00 -> 151.9 mm
- net Net-(J13-Pin_2): track 0.00 -> 105.2 mm
- net Net-(U6-B4): track 0.00 -> 102.6 mm
- net Net-(J1-Pin_2): track 0.00 -> 94.9 mm
- net Net-(J16-Pin_3): track 0.00 -> 93.5 mm
- net Net-(U6-B2): track 0.00 -> 90.8 mm
- net Net-(J15-Pin_3): track 0.00 -> 82.7 mm
- net Net-(U5-B3): track 0.00 -> 79.5 mm
- net Net-(J15-Pin_4): track 0.00 -> 79.4 mm
- net Net-(U3-17_A3_TX4_SDA1): track 0.00 -> 75.2 mm
- net Net-(U3-16_A2_RX4_SCL1): track 0.00 -> 75.2 mm
- net Net-(U5-B1): track 0.00 -> 58.1 mm
- net Net-(U5-B4): track 0.00 -> 48.5 mm
- net Net-(U5-B2): track 0.00 -> 45.7 mm
- net Net-(U4-IO33): track 0.00 -> 43.5 mm
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- added copper zone on In2.Cu, net +5V
- added copper zone on In1.Cu, net GND
Other:
- board outline added: 145 x 110 mm
- copper layers 2 -> 4
- board text added: "ProtosuitDevBoard v1.0 - 2026 lululombard Miggy"

Commit message: New shaders + credit for previous shaders
Parts:
- removed U5: Level Shifter LED matrix, Aliexpress:LEVEL_SHIFTER_TXS0108E
- removed U6: Level Shifter LED strips, Aliexpress:LEVEL_SHIFTER_TXS0108E
Connections:
- RV1 pad 2: Net-(U5-B1) -> Net-(U3-21_A7_RX5_BCLK1)
- RV2 pad 2: Net-(U5-B2) -> Net-(U3-20_A6_TX5_LRCLK1)
- RV3 pad 2: Net-(U5-B3) -> Net-(U3-6_OUT1D)
- RV4 pad 2: Net-(U5-B4) -> Net-(U3-5_IN2)
- RV5 pad 2: Net-(U6-B1) -> Net-(U4-IO5)
- RV6 pad 2: Net-(U6-B2) -> Net-(U4-IO23)
- RV7 pad 2: Net-(U6-B3) -> Net-(U4-IO19)
- RV8 pad 2: Net-(U6-B4) -> Net-(U4-IO18)
- RV9 pad 2: Net-(U6-B5) -> Net-(U4-IO26)
Routing:
- net Net-(U6-B4): track 102.6 -> 0.00 mm
- net Net-(U4-IO23): track 34.5 -> 128.8 mm
- net Net-(U3-6_OUT1D): track 37.2 -> 130.0 mm
- net Net-(U6-B2): track 90.8 -> 0.00 mm
- net Net-(U4-IO18): track 31.8 -> 116.0 mm
- net Net-(U5-B3): track 79.5 -> 0.00 mm
- net Net-(J12-Pin_2): track 151.9 -> 88.7 mm
- net Net-(U3-21_A7_RX5_BCLK1): track 27.4 -> 88.0 mm
- net Net-(U5-B1): track 58.1 -> 0.00 mm
- net Net-(U3-5_IN2): track 34.0 -> 88.9 mm
- net Net-(U5-B4): track 48.5 -> 0.00 mm
- net Net-(U5-B2): track 45.7 -> 0.00 mm
- net Net-(J13-Pin_2): track 105.2 -> 67.8 mm
- net Net-(U6-B1): track 32.9 -> 0.00 mm
- net Net-(U3-20_A6_TX5_LRCLK1): track 23.9 -> 54.2 mm
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