File: ProtosuitDevBoard/ProtosuitDevBoard.kicad_sch (KiCad schematic)
At the start: 31 parts, among them J1 XT60 IN, J10 Left Ear, J11 Right Ear, J12 Microphone input, J13 Display I2C, J14 Extra I2C, J15 Boop Sensor I2C, J16 Gyroscope I2C, J2 RPi Out, J3 Front Left, J4 Back Right, J5 Back Left, J6 Front Right, J7 Upper Arch, J8 Left Fin, J9 Right Fin, U1 DC-DC 5v 5A TPS54X60, U2 DC-DC 5v 8A CRDC2580, U3 Teensy4.0, U4 ESP32 Mini, U5 Level Shifter TXS0108E, U6 Level Shifter TXS0108E

Commit message: Final dev board
Parts:
- added J17: DHT22 sensor, Connector_JST:JST_XH_B3B-XH-A_1x03_P2.50mm_Vertical, symbol Connector_Generic:Conn_01x03
- added Q1: 2N3904, Package_TO_SOT_THT:TO-92_Inline, symbol Transistor_BJT:2N3904
- added R1: 4k7, Resistor_THT:R_Axial_DIN0207_L6.3mm_D2.5mm_P2.54mm_Vertical, symbol Device:R
- added R2: 2k2, Resistor_THT:R_Axial_DIN0207_L6.3mm_D2.5mm_P2.54mm_Vertical, symbol Device:R
- added R3: 100k, Resistor_THT:R_Axial_DIN0207_L6.3mm_D2.5mm_P2.54mm_Vertical, symbol Device:R
- added R4: 10k, Resistor_THT:R_Axial_DIN0207_L6.3mm_D2.5mm_P2.54mm_Vertical, symbol Device:R
- added U7: MPU6050 Gyroscope, Aliexpress:GYRO_MPU6050, symbol Aliexpress:GYRO_MPU6050
- J1: value XT60 IN -> PWR IN
- J16: value Gyroscope I2C -> FAN; footprint Connector_JST:JST_XH_B4B-XH-A_1x04_P2.50mm_Vertical -> Connector:FanPinHeader_1x04_P2.54mm_Vertical
- U3: value Teensy4.0 -> Teensy 4.0
- U4: value ESP32 Mini -> Wemos D1 Mini ESP32
- U5: value Level Shifter TXS0108E -> Level Shifter LED matrix
- U6: value Level Shifter TXS0108E -> Level Shifter LED strips
Connections:
- net GND: now reaches J10.1 (Pin_1), J11.1 (Pin_1), J13.1 (Pin_1), J14.1 (Pin_1), J3.1 (Pin_1), J4.1 (Pin_1), J5.1 (Pin_1), J6.1 (Pin_1), J7.1 (Pin_1), J8.1 (Pin_1), J9.1 (Pin_1), U2.4 (GND_OUT), U3.32 (GND), U4.27 (GND)
- net GND: now also J1.1 (Pin_1), J12.1 (Pin_1), J15.1 (Pin_1), J16.1 (Pin_1), J2.1 (Pin_1), U1.2 (GND_IN), U1.4 (GND_OUT), U2.2 (GND_IN), U3.1 (GND), U3.17 (GND), U3.47 (GND), U4.1 (GND), U4.2 (NC), U4.31 (GND), U5.20 (GND), U6.20 (GND), J17.1 (Pin_1), Q1.1 (E), R3.1, U7.2 (GND)
- net +5V: now reaches J10.2 (Pin_2), J11.2 (Pin_2), J3.2 (Pin_2), J4.2 (Pin_2), J5.2 (Pin_2), J6.2 (Pin_2), J7.2 (Pin_2), J8.2 (Pin_2), J9.2 (Pin_2), U2.3 (VOUT), U3.33 (VIN), U4.28 (VCC), U5.11 (VB), U6.11 (VB)
- net +5V: now also J16.2 (Pin_2), J17.2 (Pin_2), R4.1
- net at J13.2 (Pin_2), J14.2 (Pin_2), U4.18 (3.3V)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: now also R1.1
- net at U4.32 (IO27): now also J17.3 (Pin_3)
- net at U4.4 (IO35): now also J16.3 (Pin_3), R1.2
- net at U4.5 (IO33): now also R2.2
- net at J15.2 (Pin_2), U5.1 (VA): now also J12.2 (Pin_2), U3.31 (3V3), U7.1 (VCC); no longer J16.2 (Pin_2), U3.16 (3V3)
- net at J15.3 (Pin_3), U3.25 (18_A4_SDA0): now also U7.4 (SDA); no longer J16.3 (Pin_3)
- net at J15.4 (Pin_4), U3.26 (19_A5_SCL0): now also U7.3 (SCL); no longer J16.4 (Pin_4)
- net at U3.49 (3V3): no longer J12.2 (Pin_2)
- new net: Q1.2 (B), R2.1, R3.2
- new net: J16.4 (Pin_4), Q1.3 (C), R4.2
Other:
- moved on the sheet: J1, J10, J11, J12, J13, J14, J15, J2, J3, J4, J5, J6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

Commit message: New shaders + credit for previous shaders
Parts:
- removed U5: Level Shifter LED matrix, Aliexpress:LEVEL_SHIFTER_TXS0108E, symbol Aliexpress:LEVEL_SHIFTER_TXS0108E
- removed U6: Level Shifter LED strips, Aliexpress:LEVEL_SHIFTER_TXS0108E, symbol Aliexpress:LEVEL_SHIFTER_TXS0108E
Connections:
- net at RV6.2: now also U4.16 (IO23)
- net at RV5.2: now also U4.17 (IO5)
- net at U4.13 (IO26): now also RV9.2
- net at U4.14 (IO18): now also RV8.2
- net at U4.15 (IO19): now also RV7.2
- net at RV2.2: now also U3.27 (20_A6_TX5_LRCLK1)
- net at U3.28 (21_A7_RX5_BCLK1): now also RV1.2
- net at U3.7 (5_IN2): now also RV4.2
- net at U3.8 (6_OUT1D): now also RV3.2
