File: hardware/pcbs/ProtosuitDevBoard/ProtosuitDevBoard.kicad_pcb (KiCad board)
At the start: 4 copper layers, 145 x 110 mm, 36 parts, among them J1 PWR IN, J10 Left Ear, J11 Right Ear, J12 Microphone input, J13 Display I2C, J14 Extra I2C, J15 Boop Sensor I2C, J16 FAN, J17 DHT22 sensor, J2 RPi Out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

Commit message: Updated documentation
Routing:
- net Net-(J16-Pin_3): track 93.5 -> 92.6 mm
Changed lines of the file:
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@@
-	)
-	(segment
-		(start 195.24 68.38)
-		(end 194.32776 68.38)
-		(width 0.2)
-		(layer "F.Cu")
-		(net 66)
 	)
 	(segment
